Commit message: added in third actuator going to make changes to control

File: src/agbot_description/urdf/gazebo_essentials_base.xacro (robot description, xacro)
@@ -4,6 +4,6 @@
 <gazebo>
     <plugin name="gazebo_ros_control" filename="libgazebo_ros_control.so">
+      <robotParam>/agbot_description</robotParam>
       <robotNamespace>/</robotNamespace>
-      <robotParam>/agbot_description</robotParam>
       <controlPeriod>0.001</controlPeriod>
       <legacyModeNS>false</legacyModeNS>
@@ -33,4 +33,10 @@
       </plugin>
 </gazebo>
+<!-- front axle controller -->
+<!-- <Gazebo>
+  <plugin name="gazebo_ros_control" filename="libgazebo_ros_control.so">
+    <robotParam>/agbot_description</robotParam>
+  </plugin>
+</Gazebo> -->
 <!--############################# Wheel friction #########################################-->
 <xacro:macro name="wheel_friction" params="prefix ">

File: src/agbot_description/urdf/robot_base.urdf.xacro (robot description, xacro)
@@ -54,4 +54,6 @@
 <xacro:base_transmission prefix="rear_left"/>
 <xacro:base_transmission prefix="rear_right"/>
+<!-- declaring front actuator -->
+<xacro:front_transmission/>
 <!-- wheel friction -->
 <xacro:wheel_friction prefix="front_left"/>

File: src/agbot_description/urdf/robot_essentials.xacro (robot description, xacro)
@@ -113,3 +113,16 @@
 </transmission>
 </xacro:macro>
+<!-- defining front axle transmission -->
+<xacro:macro name="front_transmission">
+<transmission name="front_trans" type="SimpleTransmission">
+  <type>transmission_interface/SimpleTransmission</type>
+  <actuator name="front_motor">
+    <hardwareInterface>hardware_interface/EffortJointInterface</hardwareInterface>
+    <mechanicalReduction>1</mechanicalReduction>
+  </actuator>
+  <joint name="front_axle_joint">
+    <hardwareInterface>hardware_interface/EffortJointInterface</hardwareInterface>
+  </joint>
+</transmission>
+</xacro:macro>
 </robot>
